File: kicad/diymetro/leds.sch (KiCad schematic (older format))
At the start: 18 parts, among them U2 74LS595

Commit message: Fix 74hc595 OE pin, Fix MBT2222A symbol + footprint, Fix clock-in jack connections.
Connections:
- net +5V: no longer U2.13 (~OE)
- net GND: now also U2.13 (~OE)
Changed lines of the file:
@@
 Text HLabel 4800 3600 0    50   Input ~ 0
 RCLK
-Text HLabel 4800 3700 0    50   Input ~ 0
-+5V
 Text HLabel 5350 4700 2    50   Input ~ 0
 GND
 Text HLabel 5050 4700 0    50   Input ~ 0
 +5V
+Text HLabel 4800 3700 0    50   Input ~ 0
+GND
 $EndSCHEMATC
