File: kicad/diymetro/switches.sch (KiCad schematic (older format))
At the start: 27 parts, among them SW1 SW_SPDT_MSM, SW2 SW_SPDT_MSM, SW3 SW_SPDT_MSM, SW4 SW_SPDT_MSM, SW5 SW_SPDT_MSM, SW6 SW_SPDT_MSM, SW7 SW_SPDT_MSM, SW8 SW_SPDT_MSM, U1 74HC4051

Commit message: Update footprints for switches.
Parts:
- SW1, SW2, SW3, SW4, SW5, SW6, SW7, SW8: footprint Tomarus:SPDT_5.08mm -> Tomarus:SPDT_Switch_4.72mm
Changed lines of the file:
@@
 F 0 "SW1" H 3600 2335 50  0000 C CNN
 F 1 "SW_SPDT_MSM" H 3600 2244 50  0000 C CNN
-F 2 "Tomarus:SPDT_5.08mm" H 3600 2050 50  0001 C CNN
+F 2 "Tomarus:SPDT_Switch_4.72mm" H 3600 2050 50  0001 C CNN
 F 3 "" H 3600 2050 50  0001 C CNN
 	1    3600 2050
@@
 F 0 "SW2" H 3600 2935 50  0000 C CNN
 F 1 "SW_SPDT_MSM" H 3600 2844 50  0000 C CNN
-F 2 "Tomarus:SPDT_5.08mm" H 3600 2650 50  0001 C CNN
+F 2 "Tomarus:SPDT_Switch_4.72mm" H 3600 2650 50  0001 C CNN
 F 3 "" H 3600 2650 50  0001 C CNN
 	1    3600 2650
@@
 F 0 "SW3" H 3600 3535 50  0000 C CNN
 F 1 "SW_SPDT_MSM" H 3600 3444 50  0000 C CNN
-F 2 "Tomarus:SPDT_5.08mm" H 3600 3250 50  0001 C CNN
+F 2 "Tomarus:SPDT_Switch_4.72mm" H 3600 3250 50  0001 C CNN
 F 3 "" H 3600 3250 50  0001 C CNN
 	1    3600 3250
@@
 F 0 "SW4" H 3600 4135 50  0000 C CNN
 F 1 "SW_SPDT_MSM" H 3600 4044 50  0000 C CNN
-F 2 "Tomarus:SPDT_5.08mm" H 3600 3850 50  0001 C CNN
+F 2 "Tomarus:SPDT_Switch_4.72mm" H 3600 3850 50  0001 C CNN
 F 3 "" H 3600 3850 50  0001 C CNN
 	1    3600 3850
@@
 F 0 "SW5" H 3600 4735 50  0000 C CNN
 F 1 "SW_SPDT_MSM" H 3600 4644 50  0000 C CNN
-F 2 "Tomarus:SPDT_5.08mm" H 3600 4450 50  0001 C CNN
+F 2 "Tomarus:SPDT_Switch_4.72mm" H 3600 4450 50  0001 C CNN
 F 3 "" H 3600 4450 50  0001 C CNN
 	1    3600 4450
@@
 F 0 "SW6" H 3600 5335 50  0000 C CNN
 F 1 "SW_SPDT_MSM" H 3600 5244 50  0000 C CNN
-F 2 "Tomarus:SPDT_5.08mm" H 3600 5050 50  0001 C CNN
+F 2 "Tomarus:SPDT_Switch_4.72mm" H 3600 5050 50  0001 C CNN
 F 3 "" H 3600 5050 50  0001 C CNN
 	1    3600 5050
@@
 F 0 "SW7" H 3600 5935 50  0000 C CNN
 F 1 "SW_SPDT_MSM" H 3600 5844 50  0000 C CNN
-F 2 "Tomarus:SPDT_5.08mm" H 3600 5650 50  0001 C CNN
+F 2 "Tomarus:SPDT_Switch_4.72mm" H 3600 5650 50  0001 C CNN
 F 3 "" H 3600 5650 50  0001 C CNN
 	1    3600 5650
@@
 F 0 "SW8" H 3600 6535 50  0000 C CNN
 F 1 "SW_SPDT_MSM" H 3600 6444 50  0000 C CNN
-F 2 "Tomarus:SPDT_5.08mm" H 3600 6250 50  0001 C CNN
+F 2 "Tomarus:SPDT_Switch_4.72mm" H 3600 6250 50  0001 C CNN
 F 3 "" H 3600 6250 50  0001 C CNN
 	1    3600 6250

Commit message: Remove some unused diodes.
Parts:
- removed D3: D, Diode_SMD:D_1206_3216Metric, symbol Device:D
Connections:
- net SA: now also U1.3 (A)
Changed lines of the file:
@@
 	6700 3050 6700 3100
-$Comp
-L Device:D D?
-U 1 1 5D1A10D4
-P 5700 3600
-AR Path="/5CAA6291/5D1A10D4" Ref="D?"  Part="1"
-AR Path="/5CAE4941/5D1A10D4" Ref="D3"  Part="1"
-F 0 "D3" H 5700 3500 50  0000 C CNN
-F 1 "D" H 5700 3700 50  0000 C CNN
-F 2 "Diode_SMD:D_1206_3216Metric" H 5700 3600 50  0001 C CNN
-F 3 "~" H 5700 3600 50  0001 C CNN
-	1    5700 3600
-	1    0    0    -1
-$EndComp
 $Comp
 L Device:R R8
@@
 Text HLabel 6700 3050 1    50   Input ~ 0
 GND
-Wire Wire Line
-	5850 3600 5900 3600
-Text HLabel 5500 3600 0    50   Input ~ 0
+Text HLabel 5900 3600 0    50   Input ~ 0
 SA
-Wire Wire Line
-	5500 3600 5550 3600
 Text HLabel 5800 3800 0    50   Input ~ 0
 S0
