File: kicad/diymetro/diymetro.sch (KiCad schematic (older format))
At the start: 32 parts, among them J1 AudioJack2_SwitchT, J2 AudioJack2_SwitchT, J3 AudioJack2_SwitchT, J4 AudioJack2_SwitchT, J5 Conn_02x08_Top_Bottom, J6 AudioJack2_SwitchT, J7 ICSP, J8 SER, Q1 MMBT2222A, Q2 MMBT2222A, SW10 SW_Push, U5 ATmega328P-PU, Y1 Crystal

Commit message: Add TL072 output buffers for gate/clock/cv outputs.
Parts:
- removed D1, D2: D, Diode_SMD:D_1206_3216Metric, symbol Device:D
- removed R2: 1K, Resistor_SMD:R_1206_3216Metric, symbol Device:R
- added C10, C11, C12, C13: 100n, Capacitor_SMD:C_1206_3216Metric, symbol Device:C
- added R47, R48: 100, Resistor_SMD:R_1206_3216Metric, symbol Device:R
- added U6, U7: TL072, Package_SO:SO-8_5.3x6.2mm_P1.27mm, symbol Amplifier_Operational:TL072
- R1: value 1K -> 100
Connections:
- net ICSP_MISO is gone; now on net AP_GATE_OUT: J7.1 (Pin_1), U5.18 (PB4)
- net AP_CLK_OUT: now also U5.13 (PD7), U6.5 (+); no longer J3.T
- net AP_GATE_OUT: now also U6.3 (+); no longer J2.T
- net GND: now also C10.1, C11.1, C12.1, C13.1
- net PIN_CVOUT: now also U7.3 (+); no longer J1.T
- net -12V: now reaches J5.1 (Pin_1)
- net -12V: now also J5.2 (Pin_2), C11.2, C13.2, U6.4 (V-), U7.4 (V-)
- net +12V: now reaches J5.10 (Pin_10)
- net +12V: now also J5.9 (Pin_9), C10.2, C12.2, U6.8 (V+), U7.8 (V+)
- net at R1.1: now also J1.T; no longer U5.13 (PD7)
- net at R1.2: now also U7.1, U7.2 (-)
- new net: J2.T, R47.1
- new net: J3.T, R48.1
- new net: R47.2, U6.1, U6.2 (-)
- new net: R48.2, U6.6 (-), U6.7
- no-connect marks 14 -> 13
Other:
- moved on the sheet: C5, C6, C7, C8, C9, D14, J1, J2, J3, J4, J5, J6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

Commit message: Move gate output pin from pin12/PB4 to pin8/PB0.
Connections:
- net AP_GATE_OUT: now also U5.14 (PB0); no longer J7.1 (Pin_1), U5.18 (PB4)
- new net ICSP_MISO: J7.1 (Pin_1), U5.18 (PB4)
- no-connect marks 13 -> 12
Other:
- moved on the sheet: C5, C6, Y1
Changed lines of the file:
@@
 Text GLabel 6550 6150 2    50   Input ~ 0
 S2
-Text GLabel 8550 4500 2    50   Input ~ 0
+Text GLabel 7400 4250 2    50   Input ~ 0
 SCLK
 Text GLabel 6950 4150 2    50   Input ~ 0
@@
 	2400 6450 2300 6450
 Connection ~ 2300 6450
-Text Label 8400 4250 0    50   ~ 0
+Text Label 6550 3850 0    50   ~ 0
 AP_GATE_OUT
 Text Label 2400 3100 2    50   ~ 0
@@
 L Device:Crystal Y1
 U 1 1 5D18CF1C
-P 8550 5150
-F 0 "Y1" V 8596 5019 50  0000 R CNN
-F 1 "Crystal" V 8505 5019 50  0000 R CNN
-F 2 "Crystal:Crystal_HC49-4H_Vertical" H 8550 5150 50  0001 C CNN
-F 3 "~" H 8550 5150 50  0001 C CNN
-	1    8550 5150
+P 8100 4600
+F 0 "Y1" V 8100 4800 50  0000 R CNN
+F 1 "Crystal" V 8100 4450 50  0000 R CNN
+F 2 "Crystal:Crystal_HC49-4H_Vertical" H 8100 4600 50  0001 C CNN
+F 3 "~" H 8100 4600 50  0001 C CNN
+	1    8100 4600
 	0    -1   -1   0
 $EndComp
@@
 L Device:C C5
 U 1 1 5D19241A
-P 8800 5300
-F 0 "C5" V 8548 5300 50  0000 C CNN
-F 1 "22p" V 8639 5300 50  0000 C CNN
-F 2 "Capacitor_SMD:C_1206_3216Metric" H 8838 5150 50  0001 C CNN
-F 3 "~" H 8800 5300 50  0001 C CNN
-	1    8800 5300
+P 8350 4750
+F 0 "C5" V 8500 4750 50  0000 C CNN
+F 1 "22p" V 8600 4750 50  0000 C CNN
+F 2 "Capacitor_SMD:C_1206_3216Metric" H 8388 4600 50  0001 C CNN
+F 3 "~" H 8350 4750 50  0001 C CNN
+	1    8350 4750
 	0    1    1    0
 $EndComp
@@
 L Device:C C6
 U 1 1 5D1924D4
-P 8800 5000
-F 0 "C6" V 8548 5000 50  0000 C CNN
-F 1 "22p" V 8639 5000 50  0000 C CNN
-F 2 "Capacitor_SMD:C_1206_3216Metric" H 8838 4850 50  0001 C CNN
-F 3 "~" H 8800 5000 50  0001 C CNN
-	1    8800 5000
+P 8350 4450
+F 0 "C6" V 8098 4450 50  0000 C CNN
+F 1 "22p" V 8189 4450 50  0000 C CNN
+F 2 "Capacitor_SMD:C_1206_3216Metric" H 8388 4300 50  0001 C CNN
+F 3 "~" H 8350 4450 50  0001 C CNN
+	1    8350 4450
 	0    1    1    0
 $EndComp
@@
 L power:GND #PWR?
 U 1 1 5D1941E5
-P 8950 5000
+P 8500 4450
 AR Path="/5CAA6291/5D1941E5" Ref="#PWR?"  Part="1"
 AR Path="/5D1941E5" Ref="#PWR0103"  Part="1"
-F 0 "#PWR0103" H 8950 4750 50  0001 C CNN
-F 1 "GND" V 8950 4800 50  0000 C CNN
-F 2 "" H 8950 5000 50  0001 C CNN
-F 3 "" H 8950 5000 50  0001 C CNN
-	1    8950 5000
+F 0 "#PWR0103" H 8500 4200 50  0001 C CNN
+F 1 "GND" V 8500 4250 50  0000 C CNN
+F 2 "" H 8500 4450 50  0001 C CNN
+F 3 "" H 8500 4450 50  0001 C CNN
+	1    8500 4450
 	0    -1   -1   0
 $EndComp
@@
 L power:GND #PWR?
 U 1 1 5D194250
-P 8950 5300
+P 8500 4750
 AR Path="/5CAA6291/5D194250" Ref="#PWR?"  Part="1"
 AR Path="/5D194250" Ref="#PWR0104"  Part="1"
-F 0 "#PWR0104" H 8950 5050 50  0001 C CNN
-F 1 "GND" V 8950 5100 50  0000 C CNN
-F 2 "" H 8950 5300 50  0001 C CNN
-F 3 "" H 8950 5300 50  0001 C CNN
-	1    8950 5300
+F 0 "#PWR0104" H 8500 4500 50  0001 C CNN
+F 1 "GND" V 8500 4550 50  0000 C CNN
+F 2 "" H 8500 4750 50  0001 C CNN
+F 3 "" H 8500 4750 50  0001 C CNN
+	1    8500 4750
 	0    -1   -1   0
 $EndComp
@@
 Wire Wire Line
 	6950 5350 7350 5350
-Text Label 8550 4650 0    50   ~ 0
+Text Label 7700 4350 0    50   ~ 0
 ICSP_SCK
-Text Label 8100 4150 0    50   ~ 0
+Text Label 6550 4250 0    50   ~ 0
 ICSP_MISO
 Text Label 6950 4050 0    50   ~ 0
@@
 	6850 4150 6950 4150
 Wire Wire Line
-	6550 4250 8100 4250
-Wire Wire Line
-	8100 4150 8100 4250
-Connection ~ 8100 4250
-Wire Wire Line
-	8100 4250 8400 4250
-Wire Wire Line
-	6550 4350 8300 4350
-Wire Wire Line
-	8300 4350 8300 4500
-Wire Wire Line
-	8300 4500 8550 4500
-Wire Wire Line
-	8550 4650 8300 4650
-Wire Wire Line
-	8300 4650 8300 4500
-Connection ~ 8300 4500
-NoConn ~ 6550 3850
-Wire Wire Line
-	8650 5000 8550 5000
-Wire Wire Line
-	8550 5000 8200 5000
-Wire Wire Line
-	8200 5000 8200 4450
-Wire Wire Line
-	8200 4450 6550 4450
-Connection ~ 8550 5000
-Wire Wire Line
-	6550 4550 8150 4550
-Wire Wire Line
-	8150 4550 8150 5300
-Wire Wire Line
-	8150 5300 8550 5300
-Wire Wire Line
-	8550 5300 8650 5300
-Connection ~ 8550 5300
+	8200 4450 8100 4450
+Wire Wire Line
+	8100 4750 8200 4750
 $Comp
 L Device:R R?
@@
 NoConn ~ 2400 1300
 NoConn ~ 2400 1100
+Wire Wire Line
+	6550 4350 7350 4350
+Wire Wire Line
+	7400 4250 7350 4250
+Wire Wire Line
+	7350 4250 7350 4350
+Wire Wire Line
+	7700 4350 7350 4350
+Connection ~ 7350 4350
+Wire Wire Line
+	6550 4450 8100 4450
+Connection ~ 8100 4450
+Wire Wire Line
+	8100 4750 7800 4750
+Wire Wire Line
+	7800 4750 7800 4550
+Wire Wire Line
+	7800 4550 6550 4550
+Connection ~ 8100 4750
 $EndSCHEMATC

Commit message: Move around some stuff.
Parts:
- removed D14: LED, LED_THT:LED_D3.0mm, symbol Device:LED
- removed R46: 1K, Resistor_SMD:R_1206_3216Metric, symbol Device:R
- added J9: OutputSelect, Connector_PinHeader_2.54mm:PinHeader_1x03_P2.54mm_Vertical, symbol Connector_Generic:Conn_01x03
- added U8: MCP4921-ESN, Package_SO:SOIC-8_3.9x4.9mm_P1.27mm, symbol Analog_DAC:MCP4921-ESN
Connections:
- net SER is gone; now on net RCLK: U5.16 (PB2)
- net +5V: now also U8.1 (VDD), U8.6 (VrefA)
- net CINSW: now also U5.15 (PB1); no longer U5.27 (PC4)
- net GND: now also U8.5 (~LDAC~), U8.7 (AVSS)
- net ICSP_MISO: now also U8.2 (~CS~)
- net RCLK: no longer J7.4 (Pin_4), U5.17 (PB3)
- net PIN_CVOUT renamed AP_CV_OUT
- net AP_CV_OUT: now also J9.2 (Pin_2)
- net SCLK renamed ICSP_SCK
- net ICSP_SCK: now also U8.3 (SCK)
- new net: J9.1 (Pin_1), U8.8 (VoutA)
- new net CV_POT_OUTPUT: J9.3 (Pin_3), U5.27 (PC4)
- new net ICSP_MOSI: J7.4 (Pin_4), U5.17 (PB3), U8.4 (SDI)
Other:
- moved on the sheet: J4, J6, Q1, Q2, R3, R4, R5, R6, R7
