File: kicad/diymetro/pots1.sch (KiCad schematic (older format))
At the start: 11 parts, among them U3 74HC4051

Commit message: Remove some unused diodes.
Parts:
- removed D12: D, Diode_SMD:D_1206_3216Metric, symbol Device:D
Connections:
- net AOUT: now also U3.3 (A)
Changed lines of the file:
@@
-$EndComp
-$Comp
-L Device:D D?
-U 1 1 5D16DF58
-P 2400 2300
-AR Path="/5CAA6291/5D16DF58" Ref="D?"  Part="1"
-AR Path="/5D16DF58" Ref="D?"  Part="1"
-AR Path="/5D17C7E9/5D16DF58" Ref="D12"  Part="1"
-F 0 "D12" H 2400 2200 50  0000 C CNN
-F 1 "D" H 2400 2400 50  0000 C CNN
-F 2 "Diode_SMD:D_1206_3216Metric" H 2400 2300 50  0001 C CNN
-F 3 "~" H 2400 2300 50  0001 C CNN
-	1    2400 2300
-	1    0    0    -1
 $EndComp
 $Comp
@@
 Text HLabel 2550 2700 0    50   Input ~ 0
 S2
-Text HLabel 2250 2300 0    50   Input ~ 0
+Text HLabel 2550 2300 0    50   Input ~ 0
 AOUT
 Text HLabel 2550 2900 0    50   Input ~ 0

Commit message: Swap CV pots GND vs 5V
Connections:
- net +5V: now also RV10.1, RV3.1, RV4.1, RV5.1, RV6.1, RV7.1, RV8.1, RV9.1; no longer RV10.3, RV3.3, RV4.3, RV5.3, RV6.3, RV7.3, RV8.3, RV9.3
- net GND: now also RV10.3, RV3.3, RV4.3, RV5.3, RV6.3, RV7.3, RV8.3, RV9.3; no longer RV10.1, RV3.1, RV4.1, RV5.1, RV6.1, RV7.1, RV8.1, RV9.1
Changed lines of the file:
@@
 	0    -1   -1   0
 $EndComp
-Text HLabel 5250 1450 1    50   Input ~ 0
+Text HLabel 4750 5250 3    50   Input ~ 0
 +5V
 Text Label 3250 2300 0    50   ~ 0
@@
 	5150 4950 5250 4950
 Connection ~ 5250 4550
-Text HLabel 4750 5250 3    50   Input ~ 0
+Text HLabel 5250 1450 1    50   Input ~ 0
 GND
 Text HLabel 2850 2100 1    50   Input ~ 0
