File: kicad/diymetro/gatepots.sch (KiCad schematic (older format))
At the start: 11 parts, among them U4 74HC4051

Commit message: Remove some unused diodes.
Parts:
- removed D13: D, Diode_SMD:D_1206_3216Metric, symbol Device:D
Connections:
- net GOUT: now also U4.3 (A)
Changed lines of the file:
@@
-$EndComp
-$Comp
-L Device:D D?
-U 1 1 5D17EE1D
-P 2400 2300
-AR Path="/5CAA6291/5D17EE1D" Ref="D?"  Part="1"
-AR Path="/5D17EE1D" Ref="D?"  Part="1"
-AR Path="/5D17C7E9/5D17EE1D" Ref="D?"  Part="1"
-AR Path="/5D1A807C/5D17EE1D" Ref="D13"  Part="1"
-F 0 "D13" H 2400 2200 50  0000 C CNN
-F 1 "D" H 2400 2400 50  0000 C CNN
-F 2 "Diode_SMD:D_1206_3216Metric" H 2400 2300 50  0001 C CNN
-F 3 "~" H 2400 2300 50  0001 C CNN
-	1    2400 2300
-	1    0    0    -1
 $EndComp
 $Comp
@@
 Text HLabel 2550 2700 0    50   Input ~ 0
 S2
-Text HLabel 2250 2300 0    50   Input ~ 0
+Text HLabel 2550 2300 0    50   Input ~ 0
 GOUT
 Text HLabel 2550 2900 0    50   Input ~ 0

Commit message: Change GND/5V on gate pots too, Optimize a lot of traces and vias.
Connections:
- net +5V: now also RV11.1, RV12.1, RV13.1, RV14.1, RV15.1, RV16.1, RV17.1, RV18.1; no longer RV11.3, RV12.3, RV13.3, RV14.3, RV15.3, RV16.3, RV17.3, RV18.3
- net GND: now also RV11.3, RV12.3, RV13.3, RV14.3, RV15.3, RV16.3, RV17.3, RV18.3; no longer RV11.1, RV12.1, RV13.1, RV14.1, RV15.1, RV16.1, RV17.1, RV18.1
Changed lines of the file:
@@
 	0    -1   -1   0
 $EndComp
-Text HLabel 5250 1450 1    50   Input ~ 0
+Text HLabel 4750 5250 3    50   Input ~ 0
 +5V
 Text Label 3250 2300 0    50   ~ 0
@@
 	5150 4950 5250 4950
 Connection ~ 5250 4550
-Text HLabel 4750 5250 3    50   Input ~ 0
+Text HLabel 5250 1450 1    50   Input ~ 0
 GND
 Text HLabel 2850 2100 1    50   Input ~ 0
