File: kicad/diymetro/diymetro.kicad_pcb (KiCad board)
At the start: 2 copper layers, 100 x 75 mm, 47 parts, among them J1 Conn_02x08_Top_Bottom, J10 ReverseSwitch, J11 Conn_01x04, J12 +5V, J2 CLKGATE_Pots, J3 Gate_Pots, J4 CV_Pots, J5 CLKOUT, J6 GATEOUT, J7 CVOUT, J8 LEDs, J9 Conn_01x04, U1 74HC4051, U2 74HC4051, U3 74LS594, U4 74LS165

Commit message: New schematics and boards.
Parts:
- removed A1: Arduino_Nano_v3.x, Module:Arduino_Nano
- removed J10: ReverseSwitch, Connector_PinHeader_2.54mm:PinHeader_1x01_P2.54mm_Vertical
- removed J11, J9: Conn_01x04, Connector_PinHeader_2.54mm:PinHeader_1x04_P2.54mm_Vertical
- removed J12: +5V, Connector_PinHeader_2.54mm:PinHeader_1x01_P2.54mm_Vertical
- removed REF** (x2): MountingHole_3.2mm_M3, MountingHole:MountingHole_3.2mm_M3
- added C7: 100n, Capacitor_SMD:C_1206_3216Metric, B.Cu at (197.4, 97.3)
- added C8: 100n, Capacitor_SMD:C_1206_3216Metric, B.Cu at (184.4, 102.4)
- added D10: LED, LED_THT:LED_D3.0mm, F.Cu at (199.6, 42.2)
- added D11: LED, LED_THT:LED_D3.0mm, F.Cu at (219.6, 42.2)
- added D12: D, Diode_SMD:D_1206_3216Metric, B.Cu at (159.9, 71.9)
- added D13: D, Diode_SMD:D_1206_3216Metric, B.Cu at (149.4, 82.3)
- added D14: LED, LED_THT:LED_D3.0mm, B.Cu at (209.8, 81.8)
- added D4: LED, LED_THT:LED_D3.0mm, F.Cu at (79.6, 42.2)
- added D5: LED, LED_THT:LED_D3.0mm, F.Cu at (99.6, 42.2)
- added D6: LED, LED_THT:LED_D3.0mm, F.Cu at (119.6, 42.2)
- added D7: LED, LED_THT:LED_D3.0mm, F.Cu at (139.6, 42.2)
- added D8: LED, LED_THT:LED_D3.0mm, F.Cu at (159.6, 42.2)
- added D9: LED, LED_THT:LED_D3.0mm, F.Cu at (179.6, 42.2)
- added Q1: PN2222A, Package_TO_SOT_SMD:SOT-23, B.Cu at (154.4, 123.2)
- added Q2: PN2222A, Package_TO_SOT_SMD:SOT-23, B.Cu at (150.6, 123.2)
- added R20: 1K, Resistor_SMD:R_1206_3216Metric, B.Cu at (204.5, 101.1)
- added R21: 1K, Resistor_SMD:R_1206_3216Metric, B.Cu at (204.5, 107.2)
- added R22: 1K, Resistor_SMD:R_1206_3216Metric, B.Cu at (216.9, 101.1)
- added R23: 1K, Resistor_SMD:R_1206_3216Metric, B.Cu at (216.9, 107.2)
- added R24: 220, Resistor_SMD:R_1206_3216Metric, B.Cu at (81.0, 45.2)
- added R25: 220, Resistor_SMD:R_1206_3216Metric, B.Cu at (100.8, 45.2)
- added R26: 220, Resistor_SMD:R_1206_3216Metric, B.Cu at (120.9, 45.2)
- added R27: 220, Resistor_SMD:R_1206_3216Metric, B.Cu at (140.9, 45.2)
- added R28: 220, Resistor_SMD:R_1206_3216Metric, B.Cu at (160.8, 45.2)
- added R29: 220, Resistor_SMD:R_1206_3216Metric, B.Cu at (180.9, 45.2)
- added R30: 220, Resistor_SMD:R_1206_3216Metric, B.Cu at (200.9, 45.2)
- added R31: 220, Resistor_SMD:R_1206_3216Metric, B.Cu at (220.9, 45.2)
- added R32: 1K, Resistor_SMD:R_1206_3216Metric, B.Cu at (213.4, 121.9)
- added R33: 1K, Resistor_SMD:R_1206_3216Metric, B.Cu at (217.8, 120.0)
- added R34: 1K, Resistor_SMD:R_1206_3216Metric, B.Cu at (217.8, 117.5)
- added R35: 1K, Resistor_SMD:R_1206_3216Metric, B.Cu at (224.2, 120.0)
- added R36: 1K, Resistor_SMD:R_1206_3216Metric, B.Cu at (224.2, 122.6)
- added R37: 1K, Resistor_SMD:R_1206_3216Metric, B.Cu at (224.2, 125.1)
- added R38: 1K, Resistor_SMD:R_1206_3216Metric, B.Cu at (224.2, 127.6)
- added R39: 1K, Resistor_SMD:R_1206_3216Metric, B.Cu at (224.2, 130.2)
- added R40: 1K, Resistor_SMD:R_1206_3216Metric, B.Cu at (224.2, 132.7)
- added R41: 1K, Resistor_SMD:R_1206_3216Metric, B.Cu at (217.8, 132.7)
- added R42: 1K, Resistor_SMD:R_1206_3216Metric, B.Cu at (217.8, 130.2)
- added R43: 1K, Resistor_SMD:R_1206_3216Metric, B.Cu at (217.8, 127.6)
- added R44: 1K, Resistor_SMD:R_1206_3216Metric, B.Cu at (217.8, 125.1)
- added R45: 10k, Resistor_SMD:R_1206_3216Metric, B.Cu at (165.4, 115.8)
- added R46: 1K, Resistor_SMD:R_1206_3216Metric, B.Cu at (210.9, 85.6)
- added RV1: R_POT, Potentiometer_THT:Potentiometer_Alps_RK09K_Single_Vertical, F.Cu at (183.3, 132.7)
- added RV10: R_POT, Potentiometer_THT:Potentiometer_Alps_RK09K_Single_Vertical, F.Cu at (223.3, 66.8)
- added RV11: R_POT, Potentiometer_THT:Potentiometer_Alps_RK09K_Single_Vertical, F.Cu at (83.3, 88.7)
- added RV12: R_POT, Potentiometer_THT:Potentiometer_Alps_RK09K_Single_Vertical, F.Cu at (103.4, 88.7)
- added RV13: R_POT, Potentiometer_THT:Potentiometer_Alps_RK09K_Single_Vertical, F.Cu at (123.3, 88.7)
- added RV14: R_POT, Potentiometer_THT:Potentiometer_Alps_RK09K_Single_Vertical, F.Cu at (143.3, 88.7)
- added RV15: R_POT, Potentiometer_THT:Potentiometer_Alps_RK09K_Single_Vertical, F.Cu at (163.3, 88.7)
- added RV16: R_POT, Potentiometer_THT:Potentiometer_Alps_RK09K_Single_Vertical, F.Cu at (183.3, 88.7)
- added RV17: R_POT, Potentiometer_THT:Potentiometer_Alps_RK09K_Single_Vertical, F.Cu at (203.3, 88.7)
- added RV18: R_POT, Potentiometer_THT:Potentiometer_Alps_RK09K_Single_Vertical, F.Cu at (223.3, 88.7)
- added RV2: R_POT, Potentiometer_THT:Potentiometer_Alps_RK09K_Single_Vertical, F.Cu at (203.4, 132.7)
- added RV3: R_POT, Potentiometer_THT:Potentiometer_Alps_RK09K_Single_Vertical, F.Cu at (83.3, 66.8)
- added RV4: R_POT, Potentiometer_THT:Potentiometer_Alps_RK09K_Single_Vertical, F.Cu at (103.4, 66.8)
- added RV5: R_POT, Potentiometer_THT:Potentiometer_Alps_RK09K_Single_Vertical, F.Cu at (123.3, 66.8)
- added RV6: R_POT, Potentiometer_THT:Potentiometer_Alps_RK09K_Single_Vertical, F.Cu at (143.4, 66.8)
- added RV7: R_POT, Potentiometer_THT:Potentiometer_Alps_RK09K_Single_Vertical, F.Cu at (163.3, 66.8)
- added RV8: R_POT, Potentiometer_THT:Potentiometer_Alps_RK09K_Single_Vertical, F.Cu at (183.3, 66.8)
- added RV9: R_POT, Potentiometer_THT:Potentiometer_Alps_RK09K_Single_Vertical, F.Cu at (203.4, 66.8)
- added SW1: SW_SPDT_MSM, Tomarus:SPDT_Switch_4.72mm, F.Cu at (80.8, 104.1)
- added SW10: SW_Push, Button_Switch_THT:SW_PUSH_6mm, B.Cu at (173.5, 118.4)
- added SW2: SW_SPDT_MSM, Tomarus:SPDT_Switch_4.72mm, F.Cu at (100.8, 104.1)
- added SW3: SW_SPDT_MSM, Tomarus:SPDT_Switch_4.72mm, F.Cu at (120.8, 104.1)
- added SW4: SW_SPDT_MSM, Tomarus:SPDT_Switch_4.72mm, F.Cu at (140.8, 104.1)
- added SW5: SW_SPDT_MSM, Tomarus:SPDT_Switch_4.72mm, F.Cu at (160.8, 104.1)
- added SW6: SW_SPDT_MSM, Tomarus:SPDT_Switch_4.72mm, F.Cu at (180.8, 104.1)
- added SW7: SW_SPDT_MSM, Tomarus:SPDT_Switch_4.72mm, F.Cu at (200.9, 104.1)
- added SW8: SW_SPDT_MSM, Tomarus:SPDT_Switch_4.72mm, F.Cu at (220.8, 104.1)
- added SW9: SW_Rotary12, Tomarus:SR2612F_RotarySwitch, F.Cu at (220.8, 125.2)
- added U5: ATmega328P-PU, Package_DIP:DIP-28_W7.62mm, B.Cu at (187.0, 118.8)
- added Y1: Crystal, Crystal:Crystal_HC49-4H_Vertical, B.Cu at (182.1, 93.5)
- C1, C3: value 220n -> 100n; footprint Capacitor_THT:C_Rect_L7.0mm_W3.5mm_P5.00mm -> Capacitor_SMD:C_1206_3216Metric; moved to B.Cu
- C2, C4: footprint Capacitor_THT:C_Disc_D4.3mm_W1.9mm_P5.00mm -> Capacitor_SMD:C_1206_3216Metric; moved to B.Cu
- C5, C6: value 100n -> 22p; footprint Capacitor_THT:C_Disc_D4.3mm_W1.9mm_P5.00mm -> Capacitor_SMD:C_1206_3216Metric; moved to B.Cu
- D1, D2, D3: footprint Diode_THT:D_DO-34_SOD68_P7.62mm_Horizontal -> Diode_SMD:D_1206_3216Metric; moved to B.Cu
- J1: value Conn_02x08_Top_Bottom -> AudioJack2_SwitchT; footprint Connector_PinHeader_2.54mm:PinHeader_2x08_P2.54mm_Vertical -> Connector_Audio:Jack_3.5mm_QingPu_WQP-PJ398SM_Vertical_CircularHoles
- J2: value CLKGATE_Pots -> AudioJack2_SwitchT; footprint Connector_PinHeader_2.54mm:PinHeader_1x02_P2.54mm_Vertical -> Connector_Audio:Jack_3.5mm_QingPu_WQP-PJ398SM_Vertical_CircularHoles
- J3: value Gate_Pots -> AudioJack2_SwitchT; footprint Connector_PinHeader_2.54mm:PinHeader_1x08_P2.54mm_Vertical -> Connector_Audio:Jack_3.5mm_QingPu_WQP-PJ398SM_Vertical_CircularHoles
- J4: value CV_Pots -> AudioJack2_SwitchT; footprint Connector_PinHeader_2.54mm:PinHeader_1x08_P2.54mm_Vertical -> Connector_Audio:Jack_3.5mm_QingPu_WQP-PJ398SM_Vertical_CircularHoles
- J5: value CLKOUT -> Conn_02x08_Top_Bottom; footprint Connector_PinHeader_2.54mm:PinHeader_1x01_P2.54mm_Vertical -> Connector_IDC:IDC-Header_2x08_P2.54mm_Vertical; moved to B.Cu
- J6: value GATEOUT -> AudioJack2_SwitchT; footprint Connector_PinHeader_2.54mm:PinHeader_1x01_P2.54mm_Vertical -> Connector_Audio:Jack_3.5mm_QingPu_WQP-PJ398SM_Vertical_CircularHoles
- J7: value CVOUT -> ICSP; footprint Connector_PinHeader_2.54mm:PinHeader_1x01_P2.54mm_Vertical -> Connector_PinHeader_2.54mm:PinHeader_2x03_P2.54mm_Vertical; moved to B.Cu
- J8: value LEDs -> SER; footprint Connector_PinHeader_2.54mm:PinHeader_1x08_P2.54mm_Vertical -> Connector_PinHeader_2.54mm:PinHeader_1x02_P2.54mm_Vertical; moved to B.Cu
- R1, R2, R3: footprint Resistor_THT:R_Axial_DIN0207_L6.3mm_D2.5mm_P7.62mm_Horizontal -> Resistor_SMD:R_1206_3216Metric; moved to B.Cu
- R10, R11, R8, R9: value 220 -> 1K; footprint Resistor_THT:R_Axial_DIN0207_L6.3mm_D2.5mm_P7.62mm_Horizontal -> Resistor_SMD:R_1206_3216Metric; moved to B.Cu
- R12, R13, R14, R15, R16, R17, R18, R19: value 10K -> 1K; footprint Resistor_THT:R_Axial_DIN0207_L6.3mm_D2.5mm_P7.62mm_Horizontal -> Resistor_SMD:R_1206_3216Metric; moved to B.Cu
- R4, R7: value 220 -> 100K; footprint Resistor_THT:R_Axial_DIN0207_L6.3mm_D2.5mm_P7.62mm_Horizontal -> Resistor_SMD:R_1206_3216Metric; moved to B.Cu
- R5: value 220 -> 10K; footprint Resistor_THT:R_Axial_DIN0207_L6.3mm_D2.5mm_P7.62mm_Horizontal -> Resistor_SMD:R_1206_3216Metric; moved to B.Cu
- R6: value 220 -> 1M; footprint Resistor_THT:R_Axial_DIN0207_L6.3mm_D2.5mm_P7.62mm_Horizontal -> Resistor_SMD:R_1206_3216Metric; moved to B.Cu
- U1: footprint Package_DIP:DIP-16_W7.62mm -> Package_SO:SOP-16_4.4x10.4mm_P1.27mm; moved to B.Cu
- U2: value 74HC4051 -> 74LS595; footprint Package_DIP:DIP-16_W7.62mm -> Package_SO:SOP-16_4.4x10.4mm_P1.27mm; moved to B.Cu
- U3: value 74LS594 -> 74HC4051; footprint Package_DIP:DIP-16_W7.62mm -> Package_SO:SOP-16_4.4x10.4mm_P1.27mm; moved to B.Cu
- U4: value 74LS165 -> 74HC4051; footprint Package_DIP:DIP-16_W7.62mm -> Package_SO:SOP-16_4.4x10.4mm_P1.27mm; moved to B.Cu
- moved J8 104.1 mm to (184.2, 113.8), turned to 180 degrees
- moved D3 95.1 mm to (189.7, 122.9)
- moved R4 82.8 mm to (155.2, 128.8), turned to 270 degrees
- moved R6 80.8 mm to (146.6, 128.8)
- moved R5 80.8 mm to (149.4, 128.8)
- moved R7 78.5 mm to (146.6, 122.9)
- moved C5 74.8 mm to (172.7, 90.7)
- moved C2 74.7 mm to (141.9, 48.5), turned to 0 degrees
- moved U2 70.8 mm to (150.9, 45.2), turned to 270 degrees
- moved D1 69.3 mm to (87.6, 131.6), turned to 0 degrees
- moved J1 69.2 mm to (120.8, 118.8)
- moved J7 63.8 mm to (213.4, 94.7), turned to 90 degrees
- moved R3 61.3 mm to (152.4, 128.8), turned to 90 degrees
- moved R19 61.2 mm to (176.8, 107.2)
- moved C6 61.1 mm to (172.7, 96.5), turned to 90 degrees
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Connections:
- C1 pad 1: Net-(A1-Pad21) -> GND
- C1 pad 2: GND -> +5V
- C3 pad 1: Net-(C3-Pad1) -> GND
- C3 pad 2: GND -> +5V
- C5 pad 2: +5V -> Net-(C5-Pad2)
- C6 pad 1: +5V -> GND
- C6 pad 2: GND -> Net-(C6-Pad2)
- D1 pad 1: Net-(D1-Pad1) -> /AP_CLK_OUT
- D1 pad 2: Net-(C3-Pad1) -> Net-(D1-Pad2)
- D2 pad 1: Net-(D2-Pad1) -> /AP_GATE_OUT
- D3 pad 1: Net-(D3-Pad1) -> SA
- J5 pad 1: Net-(D2-Pad1) -> Net-(J5-Pad1)
- J7 pad 1: Net-(D1-Pad1) -> /ICSP_MISO
- R1 pad 2: Net-(D2-Pad2) -> Net-(D1-Pad2)
- R10 pad 1: Net-(R10-Pad1) -> /Switches/SW1
- R10 pad 2: Net-(J8-Pad7) -> Net-(R10-Pad2)
- R11 pad 1: Net-(R11-Pad1) -> GND
- R11 pad 2: Net-(J8-Pad8) -> /Switches/SW1
- R12 pad 1: Net-(J9-Pad1) -> /Switches/SW2
- R12 pad 2: GND -> Net-(R12-Pad2)
- R13 pad 1: Net-(J9-Pad2) -> GND
- R13 pad 2: GND -> /Switches/SW2
- R14 pad 1: Net-(J9-Pad3) -> /Switches/SW3
- R14 pad 2: GND -> Net-(R14-Pad2)
- R15 pad 1: Net-(J9-Pad4) -> GND
- R15 pad 2: GND -> /Switches/SW3
- R16 pad 1: Net-(J11-Pad1) -> /Switches/SW4
- R16 pad 2: GND -> Net-(R16-Pad2)
- R17 pad 1: Net-(J11-Pad2) -> GND
- R17 pad 2: GND -> /Switches/SW4
- R18 pad 1: Net-(J11-Pad3) -> /Switches/SW5
- R18 pad 2: GND -> Net-(R18-Pad2)
- R19 pad 1: Net-(J11-Pad4) -> GND
- R19 pad 2: GND -> /Switches/SW5
- R2 pad 1: Net-(A1-Pad6) -> /ICSP_MISO
- R2 pad 2: Net-(D3-Pad2) -> Net-(D2-Pad2)
- R3 pad 1: GND -> +5V
- R3 pad 2: Net-(A1-Pad16) -> /AP_RST_IN
- R4 pad 1: Net-(R4-Pad1) -> Net-(Q1-Pad2)
- R4 pad 2: Net-(J8-Pad1) -> Net-(J4-PadT)
- R5 pad 1: Net-(R5-Pad1) -> +5V
- R5 pad 2: Net-(J8-Pad2) -> /AP_CLK_IN
- R6 pad 1: Net-(R6-Pad1) -> +5V
- R6 pad 2: Net-(J8-Pad3) -> CINSW
- R7 pad 1: Net-(R7-Pad1) -> Net-(Q2-Pad2)
- R7 pad 2: Net-(J8-Pad4) -> Net-(J6-PadTN)
- R8 pad 1: Net-(R8-Pad1) -> /Switches/SW0
- R8 pad 2: Net-(J8-Pad5) -> Net-(R8-Pad2)
- R9 pad 1: Net-(R9-Pad1) -> GND
- R9 pad 2: Net-(J8-Pad6) -> /Switches/SW0
- U1 pad 1: Net-(J3-Pad5) -> /Switches/SW4
- U1 pad 12: Net-(J3-Pad4) -> /Switches/SW3
- U1 pad 13: Net-(J3-Pad1) -> /Switches/SW0
- U1 pad 14: Net-(J3-Pad2) -> /Switches/SW1
- U1 pad 15: Net-(J3-Pad3) -> /Switches/SW2
- U1 pad 2: Net-(J3-Pad7) -> /Switches/SW6
- U1 pad 3: Net-(A1-Pad21) -> Net-(D3-Pad2)
- U1 pad 4: Net-(J3-Pad8) -> /Switches/SW7
- U1 pad 5: Net-(J3-Pad6) -> /Switches/SW5
- U2 pad 1: Net-(J4-Pad5) -> Net-(R25-Pad1)
- U2 pad 10: S1 -> +5V
- U2 pad 11: S0 -> SCLK
- U2 pad 12: Net-(J4-Pad4) -> RCLK
- U2 pad 13: Net-(J4-Pad1) -> +5V
- U2 pad 14: Net-(J4-Pad2) -> SER
- U2 pad 15: Net-(J4-Pad3) -> Net-(R24-Pad1)
- U2 pad 2: Net-(J4-Pad7) -> Net-(R26-Pad1)
- U2 pad 3: Net-(C3-Pad1) -> Net-(R27-Pad1)
- U2 pad 4: Net-(J4-Pad8) -> Net-(R28-Pad1)
- U2 pad 5: Net-(J4-Pad6) -> Net-(R29-Pad1)
- U2 pad 6: GND -> Net-(R30-Pad1)
- U2 pad 7: GND -> Net-(R31-Pad1)
- U2 pad 9: S2 -> Net-(U2-Pad9)
- U3 pad 1: Net-(R5-Pad1) -> /CV Pots/A4
- U3 pad 10: +5V -> S1
- U3 pad 11: SCLK -> S0
- U3 pad 12: RCLK -> /CV Pots/A3
- U3 pad 13: +5V -> /CV Pots/A0
- U3 pad 14: SER -> /CV Pots/A1
- U3 pad 15: Net-(R4-Pad1) -> /CV Pots/A2
- U3 pad 2: Net-(R6-Pad1) -> /CV Pots/A6
- U3 pad 3: Net-(R7-Pad1) -> Net-(D12-Pad2)
- U3 pad 4: Net-(R8-Pad1) -> /CV Pots/A7
- U3 pad 5: Net-(R9-Pad1) -> /CV Pots/A5
- U3 pad 6: Net-(R10-Pad1) -> GND
- U3 pad 7: Net-(R11-Pad1) -> GND
- U3 pad 9: Net-(U3-Pad9) -> S2
- U4 pad 1: Net-(U4-Pad1) -> /Gate Pots/GA4
- U4 pad 10: Net-(U4-Pad10) -> S1
- U4 pad 11: Net-(J11-Pad4) -> S0
- U4 pad 12: Net-(J11-Pad3) -> /Gate Pots/GA3
- U4 pad 13: Net-(J11-Pad2) -> /Gate Pots/GA0
- U4 pad 14: Net-(J11-Pad1) -> /Gate Pots/GA1
- U4 pad 15: CE -> /Gate Pots/GA2
- U4 pad 2: CP -> /Gate Pots/GA6
- U4 pad 3: Net-(J9-Pad4) -> Net-(D13-Pad2)
- U4 pad 4: Net-(J9-Pad3) -> /Gate Pots/GA7
- U4 pad 5: Net-(J9-Pad2) -> /Gate Pots/GA5
- U4 pad 6: Net-(J9-Pad1) -> GND
- U4 pad 7: Net-(U4-Pad7) -> GND
- U4 pad 9: QH -> S2
Routing:
- net +5V: track 229.1 -> 678.9 mm, vias 8 -> 5
- net GND: track 367.5 -> 61.4 mm, vias 2 -> 22
- net /ICSP_MISO: track 0.00 -> 219.7 mm
- net Net-(R1-Pad1): track 2.92 -> 139.9 mm, vias 0 -> 4
- net /Switches/SW7: track 0.00 -> 97.4 mm, vias 0 -> 4
- net PIN_CVOUT: track 0.00 -> 86.5 mm, vias 0 -> 3
- net /Switches/SW0: track 0.00 -> 81.7 mm, vias 0 -> 1
- net /Gate Pots/GA7: track 0.00 -> 81.6 mm, vias 0 -> 2
- net /Switches/SW6: track 0.00 -> 78.0 mm, vias 0 -> 1
- net PIN_GATEOUT: track 0.00 -> 77.7 mm
- net Net-(A1-Pad21): track 76.6 -> 0.00 mm
- net /CV Pots/A0: track 0.00 -> 73.9 mm
- net /Gate Pots/GA0: track 0.00 -> 73.4 mm
- net /CV Pots/A7: track 0.00 -> 73.0 mm, vias 0 -> 1
- net QH: track 72.5 -> 0.00 mm
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- added copper zone on F.Cu, net GND
Other:
- board size 100 x 75 mm -> 162.8 x 100 mm
- board text added: "."
- board text added: "ICSP"
- board text added: "JLCJLCJLCJLC"
- board text added: "R32-44"
- board text added: "RED STRIPE"
- board text added: "SER"
- board text added: "Tomarus Sequencer v1.0 github.com/tomarus/diymetro Inspired by Ryk & Intellijel"

Commit message: Add mains cap, Reduce font size.
Parts:
- added C9: 100uF, Tomarus:GenericCap, B.Cu at (100.8, 115.3)
Routing:
- net +5V: track 678.9 -> 688.2 mm
Changed lines of the file:
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@@
     (thickness 1.6)
     (drawings 13)
-    (tracks 967)
+    (tracks 972)
     (zones 0)
-    (modules 112)
+    (modules 113)
     (nets 113)
   )
@@
     )
   )
+  (module Tomarus:GenericCap (layer B.Cu)
+    (at 100.838 115.316)
+    (fp_text reference C9 (at 0 1.016) (layer B.SilkS)
+      (effects (font (size 1 1) (thickness 0.15)) (justify mirror))
+    )
+    (fp_text value 100uF (at 0 -3.2385) (layer B.Fab)
+      (effects (font (size 1 1) (thickness 0.15)) (justify mirror))
+    )
+    (fp_line (start -4.064 -2.286) (end 4.064 -2.286) (layer B.SilkS) (width 0.15))
+    (fp_line (start 4.064 -2.286) (end 4.064 0.254) (layer B.SilkS) (width 0.15))
+    (fp_line (start 4.064 0.254) (end -4.064 0.254) (layer B.SilkS) (width 0.15))
+    (fp_line (start -4.064 0.254) (end -4.064 -2.286) (layer B.SilkS) (width 0.15))
+    (fp_line (start 1.27 0.254) (end 1.27 -2.286) (layer B.SilkS) (width 0.15))
+    (fp_text user + (at -4.7625 -0.9525) (layer B.SilkS)
+      (effects (font (size 1 1) (thickness 0.15)) (justify mirror))
+    )
+    (pad 1 thru_hole rect (at -2.54 -1.016) (size 1.8 1.8) (drill 1) (layers *.Cu *.Mask)
+      (net 8 +5V))
+    (pad 2 thru_hole circle (at 0 -1.016) (size 1.8 1.8) (drill 1) (layers *.Cu *.Mask)
+      (net 1 GND))
+    (pad 2 thru_hole circle (at 2.54 -1.016) (size 1.8 1.8) (drill 1) (layers *.Cu *.Mask)
+      (net 1 GND))
+  )
   (gr_text ICSP (at 210.82 97.282) (layer B.SilkS)
     (effects (font (size 1 1) (thickness 0.2)) (justify mirror))
@@
   (segment (start 186.8394 103.762) (end 187.0456 103.5558) (width 0.75) (layer B.Cu) (net 8))
   (segment (start 184.404 103.762) (end 186.8394 103.762) (width 0.75) (layer B.Cu) (net 8))
+  (segment (start 93.423314 109.093) (end 92.202 109.093) (width 0.75) (layer B.Cu) (net 8))
+  (segment (start 94.741 109.093) (end 93.423314 109.093) (width 0.75) (layer B.Cu) (net 8))
+  (segment (start 98.298 112.65) (end 94.741 109.093) (width 0.75) (layer B.Cu) (net 8))
+  (segment (start 98.298 114.3) (end 98.298 112.65) (width 0.75) (layer B.Cu) (net 8))
   (segment (start 94.358 129.032) (end 94.5815 129.032) (width 0.25) (layer B.Cu) (net 9))
   (segment (start 91.818 131.572) (end 94.358 129.032) (width 0.25) (layer B.Cu) (net 9))
@@
   (segment (start 80.002 108.828) (end 80.7974 108.828) (width 0.25) (layer B.Cu) (net 86))
   (segment (start 76.962 105.788) (end 80.002 108.828) (width 0.25) (layer B.Cu) (net 86))
+  (segment (start 84.788294 110.344021) (end 97.370294 110.344021) (width 0.25) (layer F.Cu) (net 86))
+  (via (at 98.044 110.236) (size 0.8) (drill 0.4) (layers F.Cu B.Cu) (net 86))
   (segment (start 80.7974 108.828) (end 83.272273 108.828) (width 0.25) (layer F.Cu) (net 86))
-  (segment (start 93.580021 110.344021) (end 93.834001 110.598001) (width 0.25) (layer F.Cu) (net 86))
-  (segment (start 93.834001 110.598001) (end 94.234 110.998) (width 0.25) (layer F.Cu) (net 86))
-  (segment (start 84.788294 110.344021) (end 93.580021 110.344021) (width 0.25) (layer F.Cu) (net 86))
-  (via (at 94.234 110.998) (size 0.8) (drill 0.4) (layers F.Cu B.Cu) (net 86))
+  (segment (start 98.951999 111.143999) (end 98.443999 110.635999) (width 0.25) (layer B.Cu) (net 86))
+  (segment (start 97.478315 110.236) (end 98.044 110.236) (width 0.25) (layer F.Cu) (net 86))
+  (segment (start 112.776 114.808) (end 109.111999 111.143999) (width 0.25) (layer B.Cu) (net 86))
+  (segment (start 98.443999 110.635999) (end 98.044 110.236) (width 0.25) (layer B.Cu) (net 86))
+  (segment (start 97.370294 110.344021) (end 97.478315 110.236) (width 0.25) (layer F.Cu) (net 86))
+  (segment (start 148.302 114.808) (end 112.776 114.808) (width 0.25) (layer B.Cu) (net 86))
   (segment (start 83.272273 108.828) (end 84.788294 110.344021) (width 0.25) (layer F.Cu) (net 86))
-  (segment (start 94.633999 111.397999) (end 94.234 110.998) (width 0.25) (layer B.Cu) (net 86))
-  (segment (start 109.365999 111.397999) (end 94.633999 111.397999) (width 0.25) (layer B.Cu) (net 86))
-  (segment (start 112.776 114.808) (end 109.365999 111.397999) (width 0.25) (layer B.Cu) (net 86))
-  (segment (start 150.236 113.524) (end 148.952 114.808) (width 0.25) (layer B.Cu) (net 86))
-  (segment (start 150.236 112.624) (end 150.236 113.524) (width 0.25) (layer B.Cu) (net 86))
-  (segment (start 148.952 114.808) (end 112.776 114.808) (width 0.25) (layer B.Cu) (net 86))
+  (segment (start 150.236 112.874) (end 148.302 114.808) (width 0.25) (layer B.Cu) (net 86))
+  (segment (start 109.111999 111.143999) (end 98.951999 111.143999) (width 0.25) (layer B.Cu) (net 86))
+  (segment (start 150.236 112.624) (end 150.236 112.874) (width 0.25) (layer B.Cu) (net 86))
   (segment (start 104.648 102.492) (end 104.648 105.788) (width 0.25) (layer B.Cu) (net 87))
   (segment (start 101.608 108.828) (end 100.7872 108.828) (width 0.25) (layer B.Cu) (net 87))

Commit message: Fix 74hc595 OE pin, Fix MBT2222A symbol + footprint, Fix clock-in jack connections.
Parts:
- Q1, Q2: value PN2222A -> MMBT2222A; footprint Package_TO_SOT_SMD:SOT-23 -> MMBT2222A:SOT23
- moved R7 5.95 mm to (144.9, 128.7), turned to 270 degrees
- moved Q2 2.81 mm to (147.8, 123.4), turned to 180 degrees
- moved R6 1.28 mm to (147.8, 128.7)
- moved R4 1.28 mm to (156.5, 128.7)
- moved R5 1.28 mm to (150.6, 128.7)
- moved R3 1.28 mm to (153.7, 128.7)
- moved Q1 0.80 mm to (153.7, 123.4), turned to 180 degrees
Connections:
- J6 pad T: CINSW -> Net-(J6-PadT)
- J6 pad TN: Net-(J6-PadTN) -> CINSW
- Q1 pad 1: /AP_RST_IN -> Net-(Q1-Pad1)
- Q1 pad 2: Net-(Q1-Pad2) -> GND
- Q1 pad 3: GND -> /AP_RST_IN
- Q2 pad 1: /AP_CLK_IN -> Net-(Q2-Pad1)
- Q2 pad 2: Net-(Q2-Pad2) -> GND
- Q2 pad 3: GND -> /AP_CLK_IN
- R4 pad 1: Net-(Q1-Pad2) -> Net-(Q1-Pad1)
- R7 pad 1: Net-(Q2-Pad2) -> Net-(Q2-Pad1)
- R7 pad 2: Net-(J6-PadTN) -> Net-(J6-PadT)
- U2 pad 13: +5V -> GND
Routing:
- net +5V: track 688.2 -> 676.3 mm, vias 5 -> 6
- net Net-(Q2-Pad1): track 0.00 -> 5.92 mm
- net Net-(Q1-Pad2): track 5.90 -> 0.00 mm
- net Net-(J6-PadTN): track 5.88 -> 0.00 mm
- net CINSW: track 67.1 -> 72.5 mm
- net Net-(J6-PadT): track 0.00 -> 4.15 mm
- net Net-(Q2-Pad2): track 3.93 -> 0.00 mm
- net Net-(Q1-Pad1): track 0.00 -> 3.91 mm
- net GND: track 61.4 -> 63.9 mm, vias 22 -> 23
- net /AP_CLK_IN: track 68.8 -> 70.6 mm
- net /AP_RST_IN: track 49.2 -> 50.5 mm
- net Net-(J4-PadT): track 5.64 -> 4.43 mm
- net S0: track 82.0 -> 81.2 mm
Other:
- board text added: "Tomarus Sequencer v1.1-dev github.com/tomarus/diymetro Inspired by Ryk & Intellijel"
- board text removed: "Tomarus Sequencer v1.0 github.com/tomarus/diymetro Inspired by Ryk & Intellijel"

Commit message: Remove some unused diodes.
Parts:
- removed D12, D13, D3: D, Diode_SMD:D_1206_3216Metric
Connections:
- U1 pad 3: Net-(D3-Pad2) -> SA
- U3 pad 3: Net-(D12-Pad2) -> PIN_CVOUT
- U4 pad 3: Net-(D13-Pad2) -> PIN_GATEOUT
Routing:
- net Net-(D3-Pad2): track 48.9 -> 0.00 mm, vias 2 -> 0
- net SA: track 6.26 -> 54.5 mm, vias 0 -> 2
- net Net-(D12-Pad2): track 12.6 -> 0.00 mm
- net PIN_CVOUT: track 86.5 -> 94.1 mm
- net PIN_GATEOUT: track 77.7 -> 81.1 mm
- net Net-(D13-Pad2): track 3.23 -> 0.00 mm
- net /Gate Pots/GA6: track 68.5 -> 70.0 mm
- net /Gate Pots/GA7: track 81.6 -> 82.9 mm

Commit message: Swap CV pots GND vs 5V
Connections:
- RV10 pad 1: GND -> +5V
- RV10 pad 3: +5V -> GND
- RV3 pad 1: GND -> +5V
- RV3 pad 3: +5V -> GND
- RV4 pad 1: GND -> +5V
- RV4 pad 3: +5V -> GND
- RV5 pad 1: GND -> +5V
- RV5 pad 3: +5V -> GND
- RV6 pad 1: GND -> +5V
- RV6 pad 3: +5V -> GND
- RV7 pad 1: GND -> +5V
- RV7 pad 3: +5V -> GND
- RV8 pad 1: GND -> +5V
- RV8 pad 3: +5V -> GND
- RV9 pad 1: GND -> +5V
- RV9 pad 3: +5V -> GND
Routing:
- net +5V: track 676.3 -> 684.1 mm
- net GND: track 63.9 -> 69.2 mm, vias 23 -> 22
- net /CV Pots/A3: track 12.9 -> 14.2 mm

Commit message: Change GND/5V on gate pots too, Optimize a lot of traces and vias.
Connections:
- RV11 pad 1: GND -> +5V
- RV11 pad 3: +5V -> GND
- RV12 pad 1: GND -> +5V
- RV12 pad 3: +5V -> GND
- RV13 pad 1: GND -> +5V
- RV13 pad 3: +5V -> GND
- RV14 pad 1: GND -> +5V
- RV14 pad 3: +5V -> GND
- RV15 pad 1: GND -> +5V
- RV15 pad 3: +5V -> GND
- RV16 pad 1: GND -> +5V
- RV16 pad 3: +5V -> GND
- RV17 pad 1: GND -> +5V
- RV17 pad 3: +5V -> GND
- RV18 pad 1: GND -> +5V
- RV18 pad 3: +5V -> GND
Routing:
- net +5V: track 684.1 -> 714.3 mm, vias 6 -> 5
- net /Switches/SW0: track 81.4 -> 91.7 mm, vias 1 -> 0
- net PIN_CVOUT: track 94.1 -> 98.8 mm, vias 3 -> 4
- net Net-(R1-Pad1): track 139.9 -> 141.5 mm, vias 4 -> 2
- net RA: track 30.3 -> 29.0 mm
- net /Gate Pots/GA3: track 12.9 -> 14.2 mm
- net S2: track 76.0 -> 75.0 mm, vias 6 -> 4
- net S1: track 94.8 -> 94.1 mm, vias 8 -> 6
- net /Gate Pots/GA7: track 82.9 -> 83.4 mm
- net S0: track 81.2 -> 81.4 mm, vias 7 -> 5

Commit message: Optimize some more traces.
Parts:
- moved R45 13.9 mm to (170.3, 128.8), turned to 90 degrees
Routing:
- net /ICSP_MISO: track 219.7 -> 155.2 mm, vias 0 -> 4
- net +5V: track 714.3 -> 700.5 mm, vias 5 -> 3
- net /Switches/SW7: track 97.4 -> 88.5 mm, vias 4 -> 0
- net PIN_CVOUT: track 98.8 -> 94.5 mm
- net /Switches/SW6: track 78.0 -> 81.7 mm
- net Net-(R1-Pad1): track 141.5 -> 138.0 mm
- net /AP_RST_IN: track 50.5 -> 47.2 mm
- net /AP_CLK_IN: track 70.6 -> 72.6 mm
- net SA: track 54.5 -> 53.1 mm
- net GND: track 69.2 -> 68.4 mm
