File: kicad/diymetro/diymetro.kicad_pcb (KiCad board)
At the start: 2 copper layers, 162.8 x 100 mm, 110 parts, among them J1 AudioJack2_SwitchT, J2 AudioJack2_SwitchT, J3 AudioJack2_SwitchT, J4 AudioJack2_SwitchT, J5 Conn_02x08_Top_Bottom, J6 AudioJack2_SwitchT, J7 ICSP, J8 SER, Q1 MMBT2222A, Q2 MMBT2222A, SW1 SW_SPDT_MSM, SW10 SW_Push, SW2 SW_SPDT_MSM, SW3 SW_SPDT_MSM, SW4 SW_SPDT_MSM, SW5 SW_SPDT_MSM, SW6 SW_SPDT_MSM, SW7 SW_SPDT_MSM, SW8 SW_SPDT_MSM, SW9 SW_Rotary12, U1 74HC4051, U2 74LS595, U3 74HC4051, U4 74HC4051, U5 ATmega328P-PU, Y1 Crystal

Commit message: Add TL072 output buffers for gate/clock/cv outputs.
Parts:
- removed D1, D2: D, Diode_SMD:D_1206_3216Metric
- removed R2: 1K, Resistor_SMD:R_1206_3216Metric
- added C10: 100n, Capacitor_SMD:C_1206_3216Metric, B.Cu at (113.5, 128.9)
- added C11: 100n, Capacitor_SMD:C_1206_3216Metric, B.Cu at (105.5, 119.0)
- added C12: 100n, Capacitor_SMD:C_1206_3216Metric, B.Cu at (133.4, 128.9)
- added C13: 100n, Capacitor_SMD:C_1206_3216Metric, B.Cu at (125.5, 118.8)
- added R47: 100, Resistor_SMD:R_1206_3216Metric, B.Cu at (108.0, 128.9)
- added R48: 100, Resistor_SMD:R_1206_3216Metric, B.Cu at (110.8, 128.9)
- added U6: TL072, Package_SO:SO-8_5.3x6.2mm_P1.27mm, B.Cu at (110.8, 123.2)
- added U7: TL072, Package_SO:SO-8_5.3x6.2mm_P1.27mm, B.Cu at (130.8, 123.1)
- R1: value 1K -> 100
- moved R1 40.4 mm to (128.0, 128.9), turned to 90 degrees
- moved C9 2.14 mm to (102.8, 114.5)
Connections:
- J1 pad T: PIN_CVOUT -> Net-(J1-PadT)
- J2 pad T: /AP_GATE_OUT -> Net-(J2-PadT)
- J3 pad T: /AP_CLK_OUT -> Net-(J3-PadT)
- J5 pad 1: Net-(J5-Pad1) -> -12V
- J5 pad 10: Net-(J5-Pad10) -> +12V
- J5 pad 2: Net-(J5-Pad2) -> -12V
- J5 pad 9: Net-(J5-Pad9) -> +12V
- J7 pad 1: /ICSP_MISO -> /AP_GATE_OUT
- R1 pad 1: Net-(R1-Pad1) -> Net-(J1-PadT)
- U5 pad 13: Net-(R1-Pad1) -> /AP_CLK_OUT
- U5 pad 18: /ICSP_MISO -> /AP_GATE_OUT
Routing:
- net /ICSP_MISO: track 155.2 -> 0.00 mm, vias 4 -> 0
- net Net-(R1-Pad1): track 138.0 -> 0.00 mm, vias 2 -> 0
- net /AP_GATE_OUT: track 6.80 -> 131.4 mm, vias 0 -> 6
- net /AP_CLK_OUT: track 5.99 -> 106.6 mm, vias 0 -> 4
- net +12V: track 0.00 -> 71.0 mm
- net -12V: track 0.00 -> 56.6 mm
- net Net-(J3-PadT): track 0.00 -> 32.0 mm
- net GND: track 68.4 -> 78.9 mm, vias 22 -> 24
- net PIN_CVOUT: track 94.5 -> 84.4 mm
- net Net-(J2-PadT): track 0.00 -> 8.20 mm
- net Net-(R48-Pad2): track 0.00 -> 7.67 mm
- net Net-(J1-PadT): track 0.00 -> 7.28 mm
- net Net-(R47-Pad2): track 0.00 -> 4.11 mm
- net Net-(D2-Pad2): track 3.82 -> 0.00 mm
- net +5V: track 700.5 -> 703.3 mm

Commit message: Move gate output pin from pin12/PB4 to pin8/PB0.
Connections:
- J7 pad 1: /AP_GATE_OUT -> /ICSP_MISO
- U5 pad 14: Net-(U5-Pad14) -> /AP_GATE_OUT
- U5 pad 18: /AP_GATE_OUT -> /ICSP_MISO
Routing:
- net /ICSP_MISO: track 0.00 -> 22.5 mm, vias 0 -> 1
- net /AP_GATE_OUT: track 131.4 -> 115.6 mm, vias 6 -> 4

Commit message: Move around some stuff.
Parts:
- removed D14: LED, LED_THT:LED_D3.0mm
- removed R46: 1K, Resistor_SMD:R_1206_3216Metric
- added J9: OutputSelect, Connector_PinHeader_2.54mm:PinHeader_1x03_P2.54mm_Vertical, B.Cu at (212.9, 111.7)
- added U8: MCP4921-ESN, Package_SO:SOIC-8_3.9x4.9mm_P1.27mm, B.Cu at (210.6, 104.0)
Connections:
- net SCLK renamed /ICSP_SCK
- J7 pad 4: RCLK -> /ICSP_MOSI
- U2 pad 14: SER -> /ICSP_MOSI
- U3 pad 3: PIN_CVOUT -> /CV_POT_OUTPUT
- U5 pad 15: Net-(R46-Pad1) -> CINSW
- U5 pad 16: SER -> RCLK
- U5 pad 17: RCLK -> /ICSP_MOSI
- U5 pad 27: CINSW -> /CV_POT_OUTPUT
- U7 pad 3: PIN_CVOUT -> /AP_CV_OUT
Routing:
- net /ICSP_MOSI: track 0.00 -> 112.8 mm, vias 0 -> 1
- net /AP_CV_OUT: track 0.00 -> 112.0 mm, vias 0 -> 2
- net /CV_POT_OUTPUT: track 0.00 -> 107.9 mm, vias 0 -> 2
- net PIN_CVOUT: track 84.4 -> 0.00 mm, vias 4 -> 0
- net SER: track 79.1 -> 0.00 mm, vias 1 -> 0
- net CINSW: track 72.5 -> 130.1 mm, vias 0 -> 4
- net RCLK: track 96.9 -> 76.6 mm, vias 1 -> 3
- net +5V: track 703.3 -> 718.7 mm
- net Net-(R46-Pad1): track 15.0 -> 0.00 mm, vias 2 -> 0
- net /ICSP_MISO: track 22.5 -> 32.8 mm
- net Net-(J9-Pad1): track 0.00 -> 9.16 mm, vias 0 -> 1
- net /ICSP_SCK: track 99.8 -> 106.5 mm
- net Net-(D14-Pad2): track 3.81 -> 0.00 mm
- net GND: track 78.9 -> 82.6 mm
- net /Switches/SW2: track 36.0 -> 37.7 mm
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Other:
- board text added: "Q/NQ"
